File: Untitled/Untitled.sch (KiCad schematic (older format))
At the start: 15 parts

Commit message: update files
Parts:
- removed U?: AP7361C-33E, Package_TO_SOT_SMD:SOT-223-3_TabPin2, symbol Regulator_Linear:AP7361C-33E
- added U1: AP7333-33SRG-7, Package_TO_SOT_SMD:SOT-23, symbol Diodes_inc:AP7333-33SRG-7
- AE1: renamed from AE?; footprint (none) -> footprint:ACAG0801-2450Trecudedkeepout
- C1, C2, C3, C4, C5: renamed from C?; footprint (none) -> Capacitor_SMD:C_0402_1005Metric
- D1: renamed from D?; footprint (none) -> LED_SMD:LED_Kingbright_APFA3010_3x1.5mm_Horizontal
- J1: renamed from J?; footprint (none) -> footprint:CONN-USB-A-PCB-TRACES
- RN1, RN2: renamed from RN?; footprint (none) -> Resistor_SMD:R_Array_Concave_4x0402
- Y1: renamed from Y?; footprint (none) -> Crystal:Crystal_SMD_Abracon_ABM10-4Pin_2.5x2.0mm
- gave numbers to parts that had none: 3
Changed lines of the file:
@@
 $EndDescr
 $Comp
-L MCU_Espressif:ESP32-C3 U?
+L MCU_Espressif:ESP32-C3 U2
 U 1 1 5FEC9B09
 P 6100 3050
-F 0 "U?" H 6100 1361 50  0000 C CNN
+F 0 "U2" H 6100 1361 50  0000 C CNN
 F 1 "ESP32-C3" H 6100 1270 50  0000 C CNN
 F 2 "Package_DFN_QFN:QFN-32-1EP_5x5mm_P0.5mm_EP3.45x3.45mm" H 6100 1750 50  0001 C CNN
@@
 $EndComp
 $Comp
-L Regulator_Linear:AP7361C-33E U?
-U 1 1 5FECE8FB
-P 3650 1700
-F 0 "U?" H 3650 1942 50  0000 C CNN
-F 1 "AP7361C-33E" H 3650 1851 50  0000 C CNN
-F 2 "Package_TO_SOT_SMD:SOT-223-3_TabPin2" H 3650 1925 50  0001 C CIN
-F 3 "https://www.diodes.com/assets/Datasheets/AP7361C.pdf" H 3650 1650 50  0001 C CNN
-	1    3650 1700
-	1    0    0    -1
-$EndComp
-$Comp
-L Connector:USB_A J?
+L Connector:USB_A J1
 U 1 1 5FED1641
 P 2000 2600
-F 0 "J?" H 2057 3067 50  0000 C CNN
+F 0 "J1" H 2057 3067 50  0000 C CNN
 F 1 "USB_A" H 2057 2976 50  0000 C CNN
-F 2 "" H 2150 2550 50  0001 C CNN
+F 2 "footprint:CONN-USB-A-PCB-TRACES" H 2150 2550 50  0001 C CNN
 F 3 " ~" H 2150 2550 50  0001 C CNN
 	1    2000 2600
@@
 	7000 4050 7500 4050
 $Comp
-L Device:Antenna AE?
+L Device:Antenna AE1
 U 1 1 5FED282C
 P 4300 2600
-F 0 "AE?" H 4380 2589 50  0000 L CNN
+F 0 "AE1" H 4380 2589 50  0000 L CNN
 F 1 "Antenna" H 4380 2498 50  0000 L CNN
-F 2 "" H 4300 2600 50  0001 C CNN
+F 2 "footprint:ACAG0801-2450Trecudedkeepout" H 4300 2600 50  0001 C CNN
 F 3 "~" H 4300 2600 50  0001 C CNN
 	1    4300 2600
@@
 $EndComp
 $Comp
-L Device:R_Pack04 RN?
+L Device:R_Pack04 RN2
 U 1 1 5FED43D3
 P 9850 3650
-F 0 "RN?" H 10038 3696 50  0000 L CNN
+F 0 "RN2" H 10038 3696 50  0000 L CNN
 F 1 "R_Pack04" H 10038 3605 50  0000 L CNN
-F 2 "" V 10125 3650 50  0001 C CNN
+F 2 "Resistor_SMD:R_Array_Concave_4x0402" V 10125 3650 50  0001 C CNN
 F 3 "~" H 9850 3650 50  0001 C CNN
 	1    9850 3650
@@
 $EndComp
 $Comp
-L Device:R_Small R?
+L Device:R_Small R1
 U 1 1 5FED4EE2
 P 8550 3300
-F 0 "R?" H 8609 3346 50  0000 L CNN
+F 0 "R1" H 8609 3346 50  0000 L CNN
 F 1 "R_Small" H 8609 3255 50  0000 L CNN
 F 2 "" H 8550 3300 50  0001 C CNN
@@
 $EndComp
 $Comp
-L Device:C_Small C?
+L Device:C_Small C5
 U 1 1 5FED54C2
 P 9350 3300
-F 0 "C?" H 9442 3346 50  0000 L CNN
+F 0 "C5" H 9442 3346 50  0000 L CNN
 F 1 "C_Small" H 9442 3255 50  0000 L CNN
-F 2 "" H 9350 3300 50  0001 C CNN
+F 2 "Capacitor_SMD:C_0402_1005Metric" H 9350 3300 50  0001 C CNN
 F 3 "~" H 9350 3300 50  0001 C CNN
 	1    9350 3300
@@
 $EndComp
 $Comp
-L Device:LED_ARGB D?
+L Device:LED_ARGB D1
 U 1 1 5FED5B1D
 P 9400 1600
-F 0 "D?" H 9400 2097 50  0000 C CNN
+F 0 "D1" H 9400 2097 50  0000 C CNN
 F 1 "LED_ARGB" H 9400 2006 50  0000 C CNN
-F 2 "" H 9400 1550 50  0001 C CNN
+F 2 "LED_SMD:LED_Kingbright_APFA3010_3x1.5mm_Horizontal" H 9400 1550 50  0001 C CNN
 F 3 "~" H 9400 1550 50  0001 C CNN
 	1    9400 1600
@@
 	4900 2750 4900 2500
 $Comp
-L Device:Crystal_GND24_Small Y?
+L Device:Crystal_GND24_Small Y1
 U 1 1 5FED6E4B
 P 4550 3450
-F 0 "Y?" V 4596 3306 50  0000 R CNN
+F 0 "Y1" V 4596 3306 50  0000 R CNN
 F 1 "Crystal_GND24_Small" V 4505 3306 50  0000 R CNN
-F 2 "" H 4550 3450 50  0001 C CNN
+F 2 "Crystal:Crystal_SMD_Abracon_ABM10-4Pin_2.5x2.0mm" H 4550 3450 50  0001 C CNN
 F 3 "~" H 4550 3450 50  0001 C CNN
 	1    4550 3450
@@
 Connection ~ 4550 3350
 $Comp
-L Device:C_Small C?
+L Device:C_Small C2
 U 1 1 5FED960B
 P 4150 3350
-F 0 "C?" V 3921 3350 50  0000 C CNN
+F 0 "C2" V 3921 3350 50  0000 C CNN
 F 1 "C_Small" V 4012 3350 50  0000 C CNN
-F 2 "" H 4150 3350 50  0001 C CNN
+F 2 "Capacitor_SMD:C_0402_1005Metric" H 4150 3350 50  0001 C CNN
 F 3 "~" H 4150 3350 50  0001 C CNN
 	1    4150 3350
@@
 $EndComp
 $Comp
-L Device:C_Small C?
+L Device:C_Small C3
 U 1 1 5FEDA25E
 P 4150 3600
-F 0 "C?" V 3921 3600 50  0000 C CNN
+F 0 "C3" V 3921 3600 50  0000 C CNN
 F 1 "C_Small" V 4012 3600 50  0000 C CNN
-F 2 "" H 4150 3600 50  0001 C CNN
+F 2 "Capacitor_SMD:C_0402_1005Metric" H 4150 3600 50  0001 C CNN
 F 3 "~" H 4150 3600 50  0001 C CNN
 	1    4150 3600
@@
 BLSEL
 $Comp
-L power:+3V3 #PWR?
+L power:+3V3 #PWR0101
 U 1 1 5FEE2170
 P 4400 1400
-F 0 "#PWR?" H 4400 1250 50  0001 C CNN
+F 0 "#PWR0101" H 4400 1250 50  0001 C CNN
 F 1 "+3V3" H 4415 1573 50  0000 C CNN
 F 2 "" H 4400 1400 50  0001 C CNN
@@
 	3100 1700 3100 1350
 $Comp
-L power:VBUS #PWR?
+L power:VBUS #PWR0102
 U 1 1 5FEE42A2
 P 3100 1350
-F 0 "#PWR?" H 3100 1200 50  0001 C CNN
+F 0 "#PWR0102" H 3100 1200 50  0001 C CNN
 F 1 "VBUS" H 3115 1523 50  0000 C CNN
 F 2 "" H 3100 1350 50  0001 C CNN
@@
 $EndComp
 $Comp
-L power:GND #PWR?
+L power:GND #PWR0103
 U 1 1 5FEE4A34
 P 3650 2200
-F 0 "#PWR?" H 3650 1950 50  0001 C CNN
+F 0 "#PWR0103" H 3650 1950 50  0001 C CNN
 F 1 "GND" H 3655 2027 50  0000 C CNN
 F 2 "" H 3650 2200 50  0001 C CNN
@@
 	3200 1700 3100 1700
 $Comp
-L Device:C_Small C?
+L Device:C_Small C4
 U 1 1 5FEE688D
 P 4300 2000
-F 0 "C?" H 4392 2046 50  0000 L CNN
+F 0 "C4" H 4392 2046 50  0000 L CNN
 F 1 "C_Small" H 4392 1955 50  0000 L CNN
-F 2 "" H 4300 2000 50  0001 C CNN
+F 2 "Capacitor_SMD:C_0402_1005Metric" H 4300 2000 50  0001 C CNN
 F 3 "~" H 4300 2000 50  0001 C CNN
 	1    4300 2000
@@
 $EndComp
 $Comp
-L Device:C_Small C?
+L Device:C_Small C1
 U 1 1 5FEE7036
 P 3200 2000
-F 0 "C?" H 3292 2046 50  0000 L CNN
+F 0 "C1" H 3292 2046 50  0000 L CNN
 F 1 "C_Small" H 3292 1955 50  0000 L CNN
-F 2 "" H 3200 2000 50  0001 C CNN
+F 2 "Capacitor_SMD:C_0402_1005Metric" H 3200 2000 50  0001 C CNN
 F 3 "~" H 3200 2000 50  0001 C CNN
 	1    3200 2000
@@
 $EndComp
 $Comp
-L power:GND #PWR?
+L power:GND #PWR0104
 U 1 1 5FEE79EB
 P 3200 2100
-F 0 "#PWR?" H 3200 1850 50  0001 C CNN
+F 0 "#PWR0104" H 3200 1850 50  0001 C CNN
 F 1 "GND" H 3205 1927 50  0000 C CNN
 F 2 "" H 3200 2100 50  0001 C CNN
@@
 $EndComp
 $Comp
-L power:GND #PWR?
+L power:GND #PWR0105
 U 1 1 5FEE7EB6
 P 4300 2100
-F 0 "#PWR?" H 4300 1850 50  0001 C CNN
+F 0 "#PWR0105" H 4300 1850 50  0001 C CNN
 F 1 "GND" H 4305 1927 50  0000 C CNN
 F 2 "" H 4300 2100 50  0001 C CNN
@@
 $EndComp
 $Comp
-L power:GND #PWR?
+L power:GND #PWR0106
 U 1 1 5FEE82E8
 P 3750 3450
-F 0 "#PWR?" H 3750 3200 50  0001 C CNN
+F 0 "#PWR0106" H 3750 3200 50  0001 C CNN
 F 1 "GND" V 3755 3322 50  0000 R CNN
 F 2 "" H 3750 3450 50  0001 C CNN
@@
 	4550 3800 4750 3800
 $Comp
-L power:GND #PWR?
+L power:GND #PWR0107
 U 1 1 5FEEA35D
 P 4550 3950
-F 0 "#PWR?" H 4550 3700 50  0001 C CNN
+F 0 "#PWR0107" H 4550 3700 50  0001 C CNN
 F 1 "GND" H 4555 3777 50  0000 C CNN
 F 2 "" H 4550 3950 50  0001 C CNN
@@
 $EndComp
 $Comp
-L power:GND #PWR?
+L power:GND #PWR0108
 U 1 1 5FEEACDE
 P 6100 5500
-F 0 "#PWR?" H 6100 5250 50  0001 C CNN
+F 0 "#PWR0108" H 6100 5250 50  0001 C CNN
 F 1 "GND" H 6105 5327 50  0000 C CNN
 F 2 "" H 6100 5500 50  0001 C CNN
@@
 	2600 2400 2600 1900
 $Comp
-L power:VBUS #PWR?
+L power:VBUS #PWR0109
 U 1 1 5FEEDEBD
 P 2600 1900
-F 0 "#PWR?" H 2600 1750 50  0001 C CNN
+F 0 "#PWR0109" H 2600 1750 50  0001 C CNN
 F 1 "VBUS" H 2615 2073 50  0000 C CNN
 F 2 "" H 2600 1900 50  0001 C CNN
@@
 USBD-
 $Comp
-L Connector_Generic:Conn_02x05_Odd_Even J?
+L Connector_Generic:Conn_02x05_Odd_Even J2
 U 1 1 5FEEEEB6
 P 9200 5050
-F 0 "J?" H 9250 5467 50  0000 C CNN
+F 0 "J2" H 9250 5467 50  0000 C CNN
 F 1 "Conn_02x05_Odd_Even" H 9250 5376 50  0000 C CNN
 F 2 "" H 9200 5050 50  0001 C CNN
@@
 $EndComp
 $Comp
-L power:+3V3 #PWR?
+L power:+3V3 #PWR0110
 U 1 1 5FEEF743
 P 5700 1350
-F 0 "#PWR?" H 5700 1200 50  0001 C CNN
+F 0 "#PWR0110" H 5700 1200 50  0001 C CNN
 F 1 "+3V3" H 5715 1523 50  0000 C CNN
 F 2 "" H 5700 1350 50  0001 C CNN
@@
 $EndComp
 $Comp
-L power:+3V3 #PWR?
+L power:+3V3 #PWR0111
 U 1 1 5FEEFD20
 P 5800 1350
-F 0 "#PWR?" H 5800 1200 50  0001 C CNN
+F 0 "#PWR0111" H 5800 1200 50  0001 C CNN
 F 1 "+3V3" H 5815 1523 50  0000 C CNN
 F 2 "" H 5800 1350 50  0001 C CNN
@@
 $EndComp
 $Comp
-L power:+3V3 #PWR?
+L power:+3V3 #PWR0112
 U 1 1 5FEF011A
 P 6000 1350
-F 0 "#PWR?" H 6000 1200 50  0001 C CNN
+F 0 "#PWR0112" H 6000 1200 50  0001 C CNN
 F 1 "+3V3" H 6015 1523 50  0000 C CNN
 F 2 "" H 6000 1350 50  0001 C CNN
@@
 $EndComp
 $Comp
-L power:+3V3 #PWR?
+L power:+3V3 #PWR0113
 U 1 1 5FEF0A33
 P 6150 1350
-F 0 "#PWR?" H 6150 1200 50  0001 C CNN
+F 0 "#PWR0113" H 6150 1200 50  0001 C CNN
 F 1 "+3V3" H 6165 1523 50  0000 C CNN
 F 2 "" H 6150 1350 50  0001 C CNN
@@
 $EndComp
 $Comp
-L power:+3V3 #PWR?
+L power:+3V3 #PWR0114
 U 1 1 5FEF0D75
 P 6400 1350
-F 0 "#PWR?" H 6400 1200 50  0001 C CNN
+F 0 "#PWR0114" H 6400 1200 50  0001 C CNN
 F 1 "+3V3" H 6415 1523 50  0000 C CNN
 F 2 "" H 6400 1350 50  0001 C CNN
@@
 $EndComp
 $Comp
-L power:+3V3 #PWR?
+L power:+3V3 #PWR0115
 U 1 1 5FEF10CE
 P 6500 1350
-F 0 "#PWR?" H 6500 1200 50  0001 C CNN
+F 0 "#PWR0115" H 6500 1200 50  0001 C CNN
 F 1 "+3V3" H 6515 1523 50  0000 C CNN
 F 2 "" H 6500 1350 50  0001 C CNN
@@
 	9800 1600 9800 1000
 $Comp
-L power:+3V3 #PWR?
+L power:+3V3 #PWR0116
 U 1 1 5FEF258C
 P 9800 1000
-F 0 "#PWR?" H 9800 850 50  0001 C CNN
+F 0 "#PWR0116" H 9800 850 50  0001 C CNN
 F 1 "+3V3" H 9815 1173 50  0000 C CNN
 F 2 "" H 9800 1000 50  0001 C CNN
@@
 $EndComp
 $Comp
-L Device:R_Pack04 RN?
+L Device:R_Pack04 RN1
 U 1 1 5FEF30E4
 P 8750 1600
-F 0 "RN?" V 8333 1600 50  0000 C CNN
+F 0 "RN1" V 8333 1600 50  0000 C CNN
 F 1 "R_Pack04" V 8424 1600 50  0000 C CNN
-F 2 "" V 9025 1600 50  0001 C CNN
+F 2 "Resistor_SMD:R_Array_Concave_4x0402" V 9025 1600 50  0001 C CNN
 F 3 "~" H 8750 1600 50  0001 C CNN
 	1    8750 1600
@@
 Text Label 7400 2650 0    50   ~ 0
 LED_B
+$Comp
+L Diodes_inc:AP7333-33SRG-7 U1
+U 1 1 5FF1FC8E
+P 3650 1750
+F 0 "U1" H 3650 2042 50  0000 C CNN
+F 1 "AP7333-33SRG-7" H 3650 1951 50  0000 C CNN
+F 2 "Package_TO_SOT_SMD:SOT-23" H 3700 2100 50  0001 C CNN
+F 3 "" H 3900 2200 50  0001 C CNN
+	1    3650 1750
+	1    0    0    -1
+$EndComp
 $EndSCHEMATC

Commit message: morr work
Parts:
- removed RN2: R_Pack04, Resistor_SMD:R_Array_Concave_4x0402, symbol Device:R_Pack04
- added C10, C9: C_Small, Capacitor_SMD:C_0603_1608Metric, symbol Device:C_Small
- added C11, C12, C6, C7, C8: C_Small, Capacitor_SMD:C_0402_1005Metric, symbol Device:C_Small
- added L1: L_Small, Inductors_SMD:L_0402, symbol Device:L_Small
- AE1: footprint footprint:ACAG0801-2450Trecudedkeepout -> footprint:Antenna-AVX-1001312
- J2: footprint (none) -> Connector_FFC-FPC:Hirose_FH12-10S-0.5SH_1x10-1MP_P0.50mm_Horizontal
- R1: footprint (none) -> Resistor_SMD:R_0402_1005Metric
- U1: footprint Package_TO_SOT_SMD:SOT-23 -> Housings_DFN_QFN:UDFN-4_1x1mm_Pitch0.65mm
- U2: symbol MCU_Espressif:ESP32-C3 -> Untitled-rescue:ESP32-C3-MCU_Espressif
- Y1: symbol Device:Crystal_GND24_Small -> Untitled-rescue:Crystal_GND24_Small-Device
Connections:
- net labels added: GP10, GP11, GP12, GP13, GP14, GP15, URX, UTX
- wire segments 67 -> 107
Other:
- moved on the sheet: AE1, C5, R1
