File: ESPVZEPTO/ESPVZEPTO.sch (KiCad schematic (older format))
At the start: 22 parts, among them J1 USB_A, J2 Conn_02x05_Odd_Even, U1 AP7333-33SRG-7, U2 ESP32-C3, Y1 Crystal_GND24_Small

Commit message: redesigned for 4 layers
Parts:
- removed AE1: Antenna, footprint:Antenna-AVX-1001312, symbol Device:Antenna
- removed J2: Conn_02x05_Odd_Even, Connector_FFC-FPC:Hirose_FH12-10S-0.5SH_1x10-1MP_P0.50mm_Horizontal, symbol Connector_Generic:Conn_02x05_Odd_Even
- removed U1: AP7333-33SRG-7, Housings_DFN_QFN:UDFN-4_1x1mm_Pitch0.65mm, symbol Diodes_inc:AP7333-33SRG-7
- added AE1: Antenna_Shield, footprint:Antenna-AVX-1001312, symbol Device:Antenna_Shield
- added J2: Conn_01x10_MountingPin, Connector_FFC-FPC:Hirose_FH12-10S-0.5SH_1x10-1MP_P0.50mm_Horizontal, symbol Connector_Generic_MountingPin:Conn_01x10_MountingPin
- added U1: NCP115AMX330TCG, Housings_DFN_QFN:UDFN-4_1x1mm_Pitch0.65mm, symbol Diodes_inc:NCP115AMX330TCG
- C2, C3: value C_Small -> 10pF
- L1: renamed from L?; footprint (none) -> Inductors_SMD:L_0402
- Y1: value Crystal_GND24_Small -> 40Mhz
- gave numbers to parts that had none: 2
Connections:
- wire segments 107 -> 130

Commit message: small tweeks and update to pin strapping
Parts:
- added R2: R_Small, Resistor_SMD:R_0402_1005Metric, symbol Device:R_Small
Connections:
- wire segments 130 -> 126
Changed lines of the file:
@@
 	8150 1600 8550 1600
 Text Label 7400 2650 0    50   ~ 0
-LED_R
+LED_G
 Text Label 7400 2550 0    50   ~ 0
-LED_G
-Text Label 7400 2450 0    50   ~ 0
 LED_B
 Wire Wire Line
@@
 $EndComp
 Wire Wire Line
-	7000 3850 7350 3850
-Wire Wire Line
-	7350 3850 7350 3950
-Wire Wire Line
 	7350 3950 7000 3950
 Wire Wire Line
-	7350 3850 7500 3850
-Connection ~ 7350 3850
-$Comp
-L power:GND #PWR0129
-U 1 1 6003F489
-P 7500 3850
-F 0 "#PWR0129" H 7500 3600 50  0001 C CNN
-F 1 "GND" H 7505 3677 50  0000 C CNN
-F 2 "" H 7500 3850 50  0001 C CNN
-F 3 "" H 7500 3850 50  0001 C CNN
-	1    7500 3850
-	0    -1   -1   0
-$EndComp
-Wire Wire Line
 	5200 3900 4900 3900
 Wire Wire Line
 	5200 4150 4900 4150
 Wire Wire Line
+	7000 2750 7400 2750
+Wire Wire Line
+	7350 2850 7000 2850
+Wire Wire Line
+	7000 2950 7350 2950
+Text Label 7400 2750 0    50   ~ 0
+LED_R
+$Comp
+L Device:R_Small R2
+U 1 1 60A101D8
+P 7400 2150
+F 0 "R2" H 7459 2196 50  0000 L CNN
+F 1 "R_Small" H 7459 2105 50  0000 L CNN
+F 2 "Resistor_SMD:R_0402_1005Metric" H 7400 2150 50  0001 C CNN
+F 3 "~" H 7400 2150 50  0001 C CNN
+	1    7400 2150
+	1    0    0    -1
+$EndComp
+Wire Wire Line
+	7400 2050 7400 1850
+$Comp
+L power:+3V3 #PWR0129
+U 1 1 60A101E0
+P 7400 1850
+F 0 "#PWR0129" H 7400 1700 50  0001 C CNN
+F 1 "+3V3" H 7415 2023 50  0000 C CNN
+F 2 "" H 7400 1850 50  0001 C CNN
+F 3 "" H 7400 1850 50  0001 C CNN
+	1    7400 1850
+	1    0    0    -1
+$EndComp
+Wire Wire Line
+	7400 2450 7400 2250
+Wire Wire Line
 	4900 3900 4900 4150
+Wire Wire Line
+	4900 4150 4900 4550
 Connection ~ 4900 4150
-Wire Wire Line
-	4900 4150 4900 4350
-$Comp
-L power:GND #PWR0130
-U 1 1 6004743E
-P 4900 4350
-F 0 "#PWR0130" H 4900 4100 50  0001 C CNN
-F 1 "GND" H 4905 4177 50  0000 C CNN
-F 2 "" H 4900 4350 50  0001 C CNN
-F 3 "" H 4900 4350 50  0001 C CNN
-	1    4900 4350
-	1    0    0    -1
-$EndComp
-Wire Wire Line
-	7000 2750 7350 2750
-Wire Wire Line
-	7350 2750 7350 2850
-Wire Wire Line
-	7350 2850 7000 2850
-Wire Wire Line
-	7000 2950 7350 2950
-Wire Wire Line
-	7350 2950 7350 2850
-Connection ~ 7350 2850
-Wire Wire Line
-	7350 2750 7500 2750
-Connection ~ 7350 2750
 $Comp
 L power:GND #PWR?
-U 1 1 60054833
-P 7500 2750
-F 0 "#PWR?" H 7500 2500 50  0001 C CNN
-F 1 "GND" H 7505 2577 50  0000 C CNN
-F 2 "" H 7500 2750 50  0001 C CNN
-F 3 "" H 7500 2750 50  0001 C CNN
-	1    7500 2750
-	0    -1   -1   0
+U 1 1 60A21779
+P 4900 4550
+F 0 "#PWR?" H 4900 4300 50  0001 C CNN
+F 1 "GND" H 4905 4377 50  0000 C CNN
+F 2 "" H 4900 4550 50  0001 C CNN
+F 3 "" H 4900 4550 50  0001 C CNN
+	1    4900 4550
+	1    0    0    -1
 $EndComp
 $EndSCHEMATC
